Commit message: added gazebo launch file launch_sim.launch

File: description/robot_core.xacro (robot description, xacro)
@@ -19,5 +19,5 @@
     <link name="chassis">
         <visual>
-        <origin xyz="0.15 0 0.075"/>
+            <origin xyz="0.15 0 0.075"/>
             <geometry>
                 <box size="0.3 0.3 0.15"/>
@@ -85,10 +85,10 @@
         <parent link="chassis"/>
         <child link="caster_wheel"/>
-        <origin xyz="0.24 0.0 0.0"/>
+        <origin xyz="0.20 0.0 0.0"/>
     </joint>
     <link name="caster_wheel">
         <visual>
             <geometry>
-                <sphere radius="0.05"/>
+                <sphere radius="0.07"/>
             </geometry>
             <material name="black"/>
@@ -96,8 +96,8 @@
         <collision>
             <geometry>
-                <sphere radius="0.05"/>
+                <sphere radius="0.07"/>
             </geometry>
         </collision>
-        <xacro:inertial_sphere mass="0.1" radius="0.5">
+        <xacro:inertial_sphere mass="0.1" radius="0.07">
             <origin xyz="0.0 0.0 0.0" rpy="0.0 0.0 0.0"/>
         </xacro:inertial_sphere>

Commit message: updated launch files

File: description/robot_core.xacro (robot description, xacro)
@@ -10,4 +10,12 @@
     <!-- BASE -->
     <link name="base_link">
+    </link>
+    <!-- BASE_FOOTPRINT -->
+    <joint name="base_footprint_joint" type="fixed">
+        <parent link="base_link"/>
+        <child link="base_footprint"/>
+        <origin xyz="0.0 0.0 0.0" rpy="0.0 0.0 0.0"/>
+    </joint>
+    <link name="base_footprint">
     </link>
     <!-- CHASSIS -->

Commit message: re-designed middle wheel of cleanbot, and added a potentially new mesh body

File: description/robot_core.xacro (robot description, xacro)
@@ -1,4 +1,4 @@
 <?xml version="1.0"?>
-<robot xmlns:xacro="httpL//www.ros.org/wiki/xacro">
+<robot xmlns:xacro="http://www.ros.org/wiki/xacro">
     <xacro:include filename="inertial_macros.xacro"/>
     <material name="white">
@@ -20,5 +20,5 @@
     </link>
     <!-- CHASSIS -->
-    <joint name="chassis_join" type="fixed">
+    <joint name="chassis_joint" type="fixed">
         <parent link="base_link"/>
         <child link="chassis"/>
@@ -77,5 +77,5 @@
         <child link="right_wheel"/>
         <origin xyz="0.0 -0.175 0.0" rpy="${pi/2} 0.0 0.0"/>
-        <axis xyz="0.0 0.0 -1.0"/>
+        <axis xyz="0.0 0.0 1.0"/>
     </joint>
     <link name="right_wheel">
@@ -102,10 +102,11 @@
         <parent link="chassis"/>
         <child link="caster_wheel"/>
-        <origin xyz="0.20 0.0 0.0"/>
+        <origin xyz="0.25 0.0 -0.04" rpy="-${pi/2} 0 0"/>
+        <axis xyz="1.0 0 0"/>
     </joint>
     <link name="caster_wheel">
         <visual>
             <geometry>
-                <sphere radius="0.075"/>
+                <cylinder radius="0.04" length="0.0254"/>
             </geometry>
             <material name="black"/>
@@ -113,8 +114,8 @@
         <collision>
             <geometry>
-                <sphere radius="0.075"/>
+                <sphere radius="0.04"/>
             </geometry>
         </collision>
-        <xacro:inertial_sphere mass="0.1" radius="0.075">
+        <xacro:inertial_sphere mass="0.1" radius="0.04">
             <origin xyz="0.0 0.0 0.0" rpy="0.0 0.0 0.0"/>
         </xacro:inertial_sphere>
