Commit message: added ros2 gazebo_control.xacro to move robot with keyboard in gazebo

File: description/cleanbot.urdf.xacro (robot description, xacro)
@@ -2,3 +2,4 @@
 <robot xmlns:xacro="http://www.ros.org/wiki/xacro" name="cleanbot">
     <xacro:include filename="robot_core.xacro"/>
+    <xacro:include filename="gazebo_control.xacro"/>
 </robot>

File: description/robot_core.xacro (robot description, xacro)
@@ -35,4 +35,7 @@
         </xacro:inertial_box>
     </link>
+    <gazebo reference="chassis">
+        <material>Gazebo/White</material>
+    </gazebo>
     <!-- LEFT WHEEL -->
     <joint name="left_wheel_joint" type="continuous">
@@ -58,4 +61,7 @@
         </xacro:inertial_cylinder>
     </link>
+    <gazebo reference="left_wheel">
+        <material>Gazebo/Black</material>
+    </gazebo>
     <!-- RIGHT WHEEL -->
     <joint name="right_wheel_joint" type="continuous">
@@ -81,4 +87,7 @@
         </xacro:inertial_cylinder>
     </link>
+    <gazebo reference="right_wheel">
+        <material>Gazebo/Black</material>
+    </gazebo>
     <!-- CASTER WHEEL-->
     <joint name="caster_wheel_join" type="fixed">
@@ -103,3 +112,8 @@
         </xacro:inertial_sphere>
     </link>
+    <gazebo reference="caster_wheel">
+        <material>Gazebo/Black</material>
+        <mu1 value="0.001"/>
+        <mu2 value="0.001"/>
+    </gazebo>
 </robot>

Commit message: added lidar scan/data in gazebo/rviz

File: description/cleanbot.urdf.xacro (robot description, xacro)
@@ -3,3 +3,4 @@
     <xacro:include filename="robot_core.xacro"/>
     <xacro:include filename="gazebo_control.xacro"/>
+    <xacro:include filename="lidar.xacro"/>
 </robot>

File: description/robot_core.xacro (robot description, xacro)
@@ -99,5 +99,5 @@
         <visual>
             <geometry>
-                <sphere radius="0.07"/>
+                <sphere radius="0.075"/>
             </geometry>
             <material name="black"/>
@@ -105,8 +105,8 @@
         <collision>
             <geometry>
-                <sphere radius="0.07"/>
+                <sphere radius="0.075"/>
             </geometry>
         </collision>
-        <xacro:inertial_sphere mass="0.1" radius="0.07">
+        <xacro:inertial_sphere mass="0.1" radius="0.075">
             <origin xyz="0.0 0.0 0.0" rpy="0.0 0.0 0.0"/>
         </xacro:inertial_sphere>

Commit message: ros2 control modifications

File: description/cleanbot.urdf.xacro (robot description, xacro)
@@ -2,5 +2,4 @@
 <robot xmlns:xacro="http://www.ros.org/wiki/xacro" name="cleanbot">
     <xacro:include filename="robot_core.xacro"/>
-    <!-- xacro:include filename="gazebo_control.xacro"/> -->
     <xacro:include filename="lidar.xacro"/>
     <xacro:include filename="ros2_control.xacro"/>

File: description/ros2_control.xacro (robot description, xacro)
@@ -1,33 +1,35 @@
 <?xml version="1.0"?>
 <robot xmlns:xacro="http://www.ros.org/wiki/xacro" name="cleanbot">
-    <ros2_control name="CLEANBOT" type="system">
-    	<hardware>
-    		<plugin>diffdrive_arduino/DiffDriveArduino</plugin>
-			<param name="left_wheel_name">left_wheel_joint</param>
-			<param name="right_wheel_name">right_wheel_joint</param>
-			<param name="loop_rate">30</param> <!-- loop rate of pid controller -->
-			<param name="device">/dev/serial/by-path/platform-fd500000.pcie-pci-0000:01:00.0-usb-0:1.4:1.0</param>
-			<param name="baud_rate">57600</param>
-			<param name="timeout_ms">1000</param>
-			<param name="enc_counts_per_rev">3436</param> <!-- CHANGE COUNTER PER REV-->
-			<!-- add pid params if needed -->
-    	</hardware>
-    	<joint name="left_wheel_joint">
-    		<command_interface name="velocity">
-    			<param name="min">-10</param>
-    			<param name="max">10</param>
-    		</command_interface>
-    		<state_interface name="velocity"/>
-    		<state_interface name="position"/>
-    	</joint>
-    	<joint name="right_wheel_joint">
-    		<command_interface name="velocity">
-    			<param name="min">-10</param>
-    			<param name="max">10</param>
-    		</command_interface>
-    		<state_interface name="velocity"/>
-    		<state_interface name="position"/>
-    	</joint>
-    </ros2_control>
+	<xacro:unless value="$(arg sim_mode)">
+		<ros2_control name="CLEANBOT" type="system">
+			<hardware>
+				<plugin>diffdrive_arduino/DiffDriveArduino</plugin>
+				<param name="left_wheel_name">left_wheel_joint</param>
+				<param name="right_wheel_name">right_wheel_joint</param>
+				<param name="loop_rate">30</param> <!-- loop rate of pid controller -->
+				<param name="device">/dev/serial/by-path/platform-fd500000.pcie-pci-0000:01:00.0-usb-0:1.4:1.0</param>
+				<param name="baud_rate">57600</param>
+				<param name="timeout_ms">1000</param>
+				<param name="enc_counts_per_rev">1120</param> <!-- CHANGE COUNTER PER REV-->
+				<!-- add pid params if needed -->
+			</hardware>
+			<joint name="left_wheel_joint">
+				<command_interface name="velocity">
+					<param name="min">-10</param>
+					<param name="max">10</param>
+				</command_interface>
+				<state_interface name="velocity"/>
+				<state_interface name="position"/>
+			</joint>
+			<joint name="right_wheel_joint">
+				<command_interface name="velocity">
+					<param name="min">-10</param>
+					<param name="max">10</param>
+				</command_interface>
+				<state_interface name="velocity"/>
+				<state_interface name="position"/>
+			</joint>
+		</ros2_control>
+    </xacro:unless>
     <!-- <ros2_control name="GazzeboSystem" type="system">
     	<hardware>
@@ -52,8 +54,32 @@
     </ros2_control>
     -->
+	<xacro:if value="$(arg sim_mode)">
+        <ros2_control name="GazeboSystem" type="system">
+            <hardware>
+                <plugin>gazebo_ros2_control/GazeboSystem</plugin>
+            </hardware>
+            <joint name="left_wheel_joint">
+                <command_interface name="velocity">
+                    <param name="min">-10</param>
+                    <param name="max">10</param>
+                </command_interface>
+                <state_interface name="velocity"/>
+                <state_interface name="position"/>
+            </joint>
+            <joint name="right_wheel_joint">
+                <command_interface name="velocity">
+                    <param name="min">-10</param>
+                    <param name="max">10</param>
+                </command_interface>
+                <state_interface name="velocity"/>
+                <state_interface name="position"/>
+            </joint>
+        </ros2_control>
+    </xacro:if>
 	<!-- may or may not comment out -->
     <gazebo>
         <plugin name="gazebo_ros2_control" filename="libgazebo_ros2_control.so">
     		<parameters>$(find cleanbot_package)/config/my_controllers.yaml</parameters>
+			<parameters>$(find cleanbot_package)/config/gaz_ros2_ctl_use_sim.yaml</parameters>
     	</plugin>
     </gazebo>
