Commit message: added ros2_control for real robot

File: description/ros2_control.xacro (robot description, xacro)
@@ -1,5 +1,34 @@
 <?xml version="1.0"?>
 <robot xmlns:xacro="http://www.ros.org/wiki/xacro" name="cleanbot">
-    <ros2_control name="GazzeboSystem" type="system">
+    <ros2_control name="CLEANBOT" type="system">
+    	<hardware>
+    		<plugin>diffdrive_arduino/DiffDriveArduino</plugin>
+			<param name="left_wheel_name">left_wheel_joint</param>
+			<param name="right_wheel_name">right_wheel_joint</param>
+			<param name="loop_rate">30</param> <!-- loop rate of pid controller -->
+			<param name="device">/dev/serial/by-path/platform-fd500000.pcie-pci-0000:01:00.0-usb-0:1.4:1.0</param>
+			<param name="baud_rate">57600</param>
+			<param name="timeout_ms">1000</param>
+			<param name="enc_counts_per_rev">3436</param> <!-- CHANGE COUNTER PER REV-->
+			<!-- add pid params if needed -->
+    	</hardware>
+    	<joint name="left_wheel_joint">
+    		<command_interface name="velocity">
+    			<param name="min">-10</param>
+    			<param name="max">10</param>
+    		</command_interface>
+    		<state_interface name="velocity"/>
+    		<state_interface name="position"/>
+    	</joint>
+    	<joint name="right_wheel_joint">
+    		<command_interface name="velocity">
+    			<param name="min">-10</param>
+    			<param name="max">10</param>
+    		</command_interface>
+    		<state_interface name="velocity"/>
+    		<state_interface name="position"/>
+    	</joint>
+    </ros2_control>
+    <!-- <ros2_control name="GazzeboSystem" type="system">
     	<hardware>
     		<plugin>gazebo_ros2_control/GazeboSystem</plugin>
@@ -22,4 +51,6 @@
     	</joint>
     </ros2_control>
+    -->
+	<!-- may or may not comment out -->
     <gazebo>
         <plugin name="gazebo_ros2_control" filename="libgazebo_ros2_control.so">

Commit message: working teleop and lidar

File: description/ros2_control.xacro (robot description, xacro)
@@ -7,10 +7,9 @@
 				<param name="left_wheel_name">left_wheel_joint</param>
 				<param name="right_wheel_name">right_wheel_joint</param>
-				<param name="loop_rate">30</param> <!-- loop rate of pid controller -->
-				<param name="device">/dev/serial/by-path/platform-fd500000.pcie-pci-0000:01:00.0-usb-0:1.4:1.0</param>
+				<param name="loop_rate">30</param>
+				<param name="device">/dev/ttyACM0</param>
 				<param name="baud_rate">57600</param>
 				<param name="timeout_ms">1000</param>
-				<param name="enc_counts_per_rev">1120</param> <!-- CHANGE COUNTER PER REV-->
-				<!-- add pid params if needed -->
+				<param name="enc_counts_per_rev">1074</param>
 			</hardware>
 			<joint name="left_wheel_joint">
@@ -32,26 +31,4 @@
 		</ros2_control>
     </xacro:unless>
-    <!-- <ros2_control name="GazzeboSystem" type="system">
-    	<hardware>
-    		<plugin>gazebo_ros2_control/GazeboSystem</plugin>
-    	</hardware>
-    	<joint name="left_wheel_joint">
-    		<command_interface name="velocity">
-    			<param name="min">-10</param>
-    			<param name="max">10</param>
-    		</command_interface>
-    		<state_interface name="velocity"/>
-    		<state_interface name="position"/>
-    	</joint>
-    	<joint name="right_wheel_joint">
-    		<command_interface name="velocity">
-    			<param name="min">-10</param>
-    			<param name="max">10</param>
-    		</command_interface>
-    		<state_interface name="velocity"/>
-    		<state_interface name="position"/>
-    	</joint>
-    </ros2_control>
-    -->
 	<xacro:if value="$(arg sim_mode)">
         <ros2_control name="GazeboSystem" type="system">
@@ -77,5 +54,4 @@
         </ros2_control>
     </xacro:if>
-	<!-- may or may not comment out -->
     <gazebo>
         <plugin name="gazebo_ros2_control" filename="libgazebo_ros2_control.so">
